Commit message: [Urdf] fix odom error

File: my_robot_description/urdf/camera.xacro (robot description, xacro)
@@ -11,6 +11,6 @@
                 <box size="0.06 0.28 0.04"/>
             </geometry>
-            <material name="black">
-                <color rgba="0 0 0 1"/>
+            <material name="red">
+                <color rgba="1 0 0 1"/>
             </material>
         </visual>

File: my_robot_description/urdf/mobile_base.xacro (robot description, xacro)
@@ -71,3 +71,8 @@
     <origin xyz="0 0 0" rpy="0 0 0"/>
   </joint>
+  <joint name="kinect_joint" type="fixed">
+    <parent link="base_link"/>
+    <child link="camera_link"/>
+    <origin xyz="0.105 0 0.15" rpy="0 0 0"/>
+  </joint>
 </robot>

File: my_robot_description/urdf/my_robot.urdf.xacro (robot description, xacro)
@@ -2,4 +2,4 @@
 <robot name="my_robot" xmlns:xacro="http://www.ros.org/wiki/xacro">
     <xacro:include filename="mobile_base.xacro" />
-    <!-- <xacro:include filename="camera.xacro" /> -->
+    <xacro:include filename="camera.xacro" />
 </robot>

Commit message: [Description] change parameter of hardware

File: my_robot_description/urdf/camera.xacro (robot description, xacro)
@@ -4,5 +4,5 @@
         <parent link="base_link"/>
         <child link="camera_link"/>
-        <origin xyz="0.3 0 0.2" rpy="0 0 0"/>
+        <origin xyz="0 0 0.13" rpy="0 0 0"/>
     </joint>
     <link name="camera_link">

File: my_robot_description/urdf/mobile_base.xacro (robot description, xacro)
@@ -1,4 +1,4 @@
 <?xml version="1.0"?>
-<robot name="unicycle" xmlns:xacro="http://www.ros.org/wiki/xacro">
+<robot name="my_robot" xmlns:xacro="http://www.ros.org/wiki/xacro">
   <xacro:property name="base_length" value="0.3" />
   <xacro:property name="base_width" value="0.2" />
@@ -6,5 +6,4 @@
   <xacro:property name="wheel_radius" value="0.034" />
   <xacro:property name="wheel_length" value="0.025" />
-  <link name="base_footprint" />
   <link name="base_link">
     <visual>
@@ -18,9 +17,11 @@
     </visual>
   </link>
-  <joint name="base_joint" type="fixed">
-    <parent link="base_footprint" />
-    <child link="base_link" />
-    <origin xyz="0 0 0" rpy="0 0 0" />
+  <joint name="base_footprint_joint" type="fixed">
+      <parent link="base_link"/>
+      <child link="base_footprint"/>
+      <origin xyz="0 0 0" rpy="0 0 0"/>
   </joint>
+  <link name="base_footprint">
+  </link>
   <link name="left_wheel">
     <visual>
@@ -77,8 +78,3 @@
     <origin xyz="-0.105 0 0.0775" rpy="0 0 0"/>
   </joint>
-  <joint name="kinect_joint" type="fixed">
-    <parent link="base_link"/>
-    <child link="camera_link"/>
-    <origin xyz="0 0 0.13" rpy="0 0 0"/>
-  </joint>
 </robot>

Commit message: add camera_depth_frame

File: my_robot_description/urdf/camera.xacro (robot description, xacro)
@@ -35,3 +35,10 @@
     </joint>
     <link name="kinect_rgb"/>
+    <!-- Alias frame cho depthimage_to_laserscan (default output_frame_id) -->
+    <joint name="camera_depth_frame_joint" type="fixed">
+        <parent link="kinect_depth"/>
+        <child link="camera_depth_frame"/>
+        <origin xyz="0 0 0" rpy="0 0 0"/>
+    </joint>
+    <link name="camera_depth_frame"/>
 </robot>

Commit message: fix map and rviz2

File: my_robot_description/urdf/camera.xacro (robot description, xacro)
@@ -35,10 +35,3 @@
     </joint>
     <link name="kinect_rgb"/>
-    <!-- Alias frame cho depthimage_to_laserscan (default output_frame_id) -->
-    <joint name="camera_depth_frame_joint" type="fixed">
-        <parent link="kinect_depth"/>
-        <child link="camera_depth_frame"/>
-        <origin xyz="0 0 0" rpy="0 0 0"/>
-    </joint>
-    <link name="camera_depth_frame"/>
 </robot>

Commit message: fix map rviz2 error

File: my_robot_description/urdf/camera.xacro (robot description, xacro)
@@ -35,3 +35,11 @@
     </joint>
     <link name="kinect_rgb"/>
+    <!-- Frame cho depthimage_to_laserscan: parent camera_link (x=tiến) thay vì optical frame
+         để slam_toolbox nhận scan đúng hướng, không bị lệch 90 độ -->
+    <joint name="camera_depth_frame_joint" type="fixed">
+        <parent link="camera_link"/>
+        <child link="camera_depth_frame"/>
+        <origin xyz="0 0 0" rpy="0 0 0"/>
+    </joint>
+    <link name="camera_depth_frame"/>
 </robot>
