Commit message: [Change from ros control to micro ros]

File: my_robot_description/urdf/mobile_base.xacro (robot description, xacro)
@@ -1,62 +1,73 @@
 <?xml version="1.0"?>
-<robot xmlns:xacro="http://www.ros.org/wiki/xacro">
-    <xacro:property name="base_length" value="0.6" />
-    <xacro:property name="base_width" value="0.4" />
-    <xacro:property name="base_height" value="0.2" />
-    <xacro:property name="wheel_radius" value="0.1" />
-    <xacro:property name="wheel_length" value="0.05" />
-    <link name="base_footprint" />
-    <link name="base_link">
-        <visual>
-            <geometry>
-                <box size="${base_length} ${base_width} ${base_height}" />
-            </geometry>
-            <origin xyz="0 0 ${base_height / 2.0}" rpy="0 0 0" />
-            <material name="blue" />
-        </visual>
-    </link>
-    <xacro:macro name="wheel_link" params="prefix">
-        <link name="${prefix}_wheel_link">
-            <visual>
-                <geometry>
-                    <cylinder radius="${wheel_radius}" length="${wheel_length}" />
-                </geometry>
-                <origin xyz="0 0 0" rpy="${pi / 2.0} 0 0" />
-                <material name="grey" />
-            </visual>
-        </link>
-    </xacro:macro>
-    <xacro:wheel_link prefix="right" />
-    <xacro:wheel_link prefix="left" />
-    <link name="caster_wheel_link">
-        <visual>
-            <geometry>
-                <sphere radius="${wheel_radius / 2.0}" />
-            </geometry>
-            <origin xyz="0 0 0" rpy="0 0 0" />
-            <material name="grey" />
-        </visual>
-    </link>
-    <joint name="base_joint" type="fixed">
-        <parent link="base_footprint" />
-        <child link="base_link" />
-        <origin xyz="0 0 ${wheel_radius}" rpy="0 0 0"/>
-    </joint>
-    <joint name="base_right_wheel_joint" type="continuous">
-        <parent link="base_link" />
-        <child link="right_wheel_link" />
-        <origin xyz="${-base_length / 4.0} ${-(base_width + wheel_length) / 2.0} 0" rpy="0 0 0" />
-        <axis xyz="0 1 0" />
-    </joint>
-    <joint name="base_left_wheel_joint" type="continuous">
-        <parent link="base_link" />
-        <child link="left_wheel_link" />
-        <origin xyz="${-base_length / 4.0} ${(base_width + wheel_length) / 2.0} 0" rpy="0 0 0" />
-        <axis xyz="0 1 0" />
-    </joint>
-    <joint name="base_caster_wheel_joint" type="fixed">
-        <parent link="base_link" />
-        <child link="caster_wheel_link" />
-        <origin xyz="${base_length / 3.0} 0 ${-wheel_radius / 2.0}" rpy="0 0 0" />
-    </joint>
+<robot name="unicycle" xmlns:xacro="http://www.ros.org/wiki/xacro">
+  <xacro:property name="base_length" value="0.3" />
+  <xacro:property name="base_width" value="0.2" />
+  <xacro:property name="base_height" value="0.15" />
+  <xacro:property name="wheel_radius" value="0.034" />
+  <xacro:property name="wheel_length" value="0.025" />
+  <link name="base_footprint" />
+  <link name="base_link">
+    <visual>
+      <geometry>
+        <box size="${base_length} ${base_width} ${base_height}" />
+      </geometry>
+      <origin xyz="0 0 0.11" rpy="0 0 0" />
+      <material name="semi_black">
+        <color rgba="0 0 0 0.75" />
+      </material>
+    </visual>
+  </link>
+  <joint name="base_joint" type="fixed">
+    <parent link="base_footprint" />
+    <child link="base_link" />
+    <origin xyz="0 0 0" rpy="0 0 0" />
+  </joint>
+  <link name="left_wheel">
+    <visual>
+      <geometry>
+        <cylinder length="${wheel_length}" radius="${wheel_radius}" />
+      </geometry>
+      <origin xyz="0.105 0.1 0.025" rpy="1.5708 0 0" />
+      <material name="blue">
+        <color rgba="0.0 0.0 1.0 1.0" />
+      </material>
+    </visual>
+  </link>
+  <link name="right_wheel">
+    <visual>
+      <geometry>
+        <cylinder length="${wheel_length}" radius="${wheel_radius}" />
+      </geometry>
+      <origin xyz="0.105 -0.1 0.025" rpy="1.5708 0 0" />
+      <material name="blue">
+        <color rgba="0.0 0.0 1.0 1.0" />
+      </material>
+    </visual>
+  </link>
+  <link name="front_ball">
+    <visual>
+      <geometry>
+        <sphere radius="0.03" />
+      </geometry>
+      <origin xyz="-0.105 0 0.03" rpy="0 0 0" />
+      <material name="gray">
+        <color rgba="0.5 0.5 0.5 1.0" />
+      </material>
+    </visual>
+  </link>
+  <joint name="left_wheel_joint" type="fixed">
+    <parent link="base_link"/>
+    <child link="left_wheel"/>
+    <origin xyz="0 0 0" rpy="0 0 0"/>
+  </joint>
+  <joint name="right_wheel_joint" type="fixed">
+    <parent link="base_link"/>
+    <child link="right_wheel"/>
+    <origin xyz="0 0 0" rpy="0 0 0"/>
+  </joint>
+  <joint name="front_ball_joint" type="fixed">
+    <parent link="base_link"/>
+    <child link="front_ball"/>
+    <origin xyz="0 0 0" rpy="0 0 0"/>
+  </joint>
 </robot>

File: my_robot_description/urdf/my_robot.urdf.xacro (robot description, xacro)
@@ -1,7 +1,5 @@
 <?xml version="1.0"?>
 <robot name="my_robot" xmlns:xacro="http://www.ros.org/wiki/xacro">
-    <xacro:include filename="common_properties.xacro" />
     <xacro:include filename="mobile_base.xacro" />
-    <xacro:include filename="mobile_base.ros2_control.xacro" />
-    <xacro:include filename="camera.xacro" />
+    <!-- <xacro:include filename="camera.xacro" /> -->
 </robot>

Commit message: [URDF] fix base link,camera link,imu link

File: my_robot_description/urdf/mobile_base.xacro (robot description, xacro)
@@ -3,5 +3,5 @@
   <xacro:property name="base_length" value="0.3" />
   <xacro:property name="base_width" value="0.2" />
-  <xacro:property name="base_height" value="0.15" />
+  <xacro:property name="base_height" value="0.065" />
   <xacro:property name="wheel_radius" value="0.034" />
   <xacro:property name="wheel_length" value="0.025" />
@@ -12,5 +12,5 @@
         <box size="${base_length} ${base_width} ${base_height}" />
       </geometry>
-      <origin xyz="0 0 0.11" rpy="0 0 0" />
+      <origin xyz="-0.105 0 0.0775" rpy="0 0 0" /> <!--4.5cm+base_height/2= 7.75cm-->
       <material name="semi_black">
         <color rgba="0 0 0 0.75" />
@@ -28,5 +28,5 @@
         <cylinder length="${wheel_length}" radius="${wheel_radius}" />
       </geometry>
-      <origin xyz="0.105 0.1 0.025" rpy="1.5708 0 0" />
+      <origin xyz="0 0.1 0.034" rpy="1.5708 0 0" />
       <material name="blue">
         <color rgba="0.0 0.0 1.0 1.0" />
@@ -39,5 +39,5 @@
         <cylinder length="${wheel_length}" radius="${wheel_radius}" />
       </geometry>
-      <origin xyz="0.105 -0.1 0.025" rpy="1.5708 0 0" />
+      <origin xyz="0 -0.1 0.034" rpy="1.5708 0 0" />
       <material name="blue">
         <color rgba="0.0 0.0 1.0 1.0" />
@@ -50,5 +50,5 @@
         <sphere radius="0.03" />
       </geometry>
-      <origin xyz="-0.105 0 0.03" rpy="0 0 0" />
+      <origin xyz="-0.21 0 0.03" rpy="0 0 0" />
       <material name="gray">
         <color rgba="0.5 0.5 0.5 1.0" />
@@ -71,8 +71,14 @@
     <origin xyz="0 0 0" rpy="0 0 0"/>
   </joint>
+  <link name="imu_link"/>
+  <joint name="imu_joint" type="fixed">
+    <parent link="base_link"/>
+    <child link="imu_link"/>
+    <origin xyz="-0.105 0 0.0775" rpy="0 0 0"/>
+  </joint>
   <joint name="kinect_joint" type="fixed">
     <parent link="base_link"/>
     <child link="camera_link"/>
-    <origin xyz="0.105 0 0.15" rpy="0 0 0"/>
+    <origin xyz="0 0 0.13" rpy="0 0 0"/>
   </joint>
 </robot>

Commit message: fix slowly map update

File: my_robot_description/urdf/mobile_base.xacro (robot description, xacro)
@@ -6,4 +6,6 @@
   <xacro:property name="wheel_radius" value="0.034" />
   <xacro:property name="wheel_length" value="0.025" />
+  <!-- Gốc tọa độ trên mặt đất -->
+  <link name="base_footprint"/>
   <link name="base_link">
     <visual>
@@ -11,5 +13,5 @@
         <box size="${base_length} ${base_width} ${base_height}" />
       </geometry>
-      <origin xyz="-0.105 0 0.0775" rpy="0 0 0" /> <!--4.5cm+base_height/2= 7.75cm-->
+      <origin xyz="-0.105 0 0.0775" rpy="0 0 0" />
       <material name="semi_black">
         <color rgba="0 0 0 0.75" />
@@ -18,10 +20,8 @@
   </link>
   <joint name="base_footprint_joint" type="fixed">
-      <parent link="base_link"/>
-      <child link="base_footprint"/>
-      <origin xyz="0 0 0" rpy="0 0 0"/>
+    <parent link="base_footprint"/>
+    <child link="base_link"/>
+    <origin xyz="0 0 0" rpy="0 0 0"/>
   </joint>
-  <link name="base_footprint">
-  </link>
   <link name="left_wheel">
     <visual>
@@ -57,4 +57,28 @@
     </visual>
   </link>
+  <!-- Kinect Physical Link -->
+  <link name="kinect_link">
+    <visual>
+      <geometry>
+        <box size="0.06 0.28 0.04"/>
+      </geometry>
+      <origin xyz="0 0 0" rpy="0 0 0" />
+      <material name="red">
+          <color rgba="1 0 0 1"/>
+      </material>
+    </visual>
+  </link>
+  <joint name="kinect_joint" type="fixed">
+    <parent link="base_link"/>
+    <child link="kinect_link"/>
+    <origin xyz="0 0 0.13" rpy="0 0 0"/>
+  </joint>
+  <!-- Kinect Optical Frame (Z forward, X right, Y down) -->
+  <link name="kinect_depth"/>
+  <joint name="kinect_depth_joint" type="fixed">
+    <parent link="kinect_link"/>
+    <child link="kinect_depth"/>
+    <origin xyz="0 0 0" rpy="-1.5708 0 -1.5708"/>
+  </joint>
   <joint name="left_wheel_joint" type="fixed">
     <parent link="base_link"/>

File: my_robot_description/urdf/my_robot.urdf.xacro (robot description, xacro)
@@ -2,4 +2,3 @@
 <robot name="my_robot" xmlns:xacro="http://www.ros.org/wiki/xacro">
     <xacro:include filename="mobile_base.xacro" />
-    <xacro:include filename="camera.xacro" />
 </robot>

Commit message: fix wheel separation

File: my_robot_description/urdf/mobile_base.xacro (robot description, xacro)
@@ -29,5 +29,5 @@
         <cylinder length="${wheel_length}" radius="${wheel_radius}" />
       </geometry>
-      <origin xyz="0 0.1 0.034" rpy="1.5708 0 0" />
+      <origin xyz="0 0.1175 0.034" rpy="1.5708 0 0" />
       <material name="blue">
         <color rgba="0.0 0.0 1.0 1.0" />
@@ -40,5 +40,5 @@
         <cylinder length="${wheel_length}" radius="${wheel_radius}" />
       </geometry>
-      <origin xyz="0 -0.1 0.034" rpy="1.5708 0 0" />
+      <origin xyz="0 -0.1175 0.034" rpy="1.5708 0 0" />
       <material name="blue">
         <color rgba="0.0 0.0 1.0 1.0" />

Commit message: change wheel separation

File: my_robot_description/urdf/mobile_base.xacro (robot description, xacro)
@@ -29,5 +29,5 @@
         <cylinder length="${wheel_length}" radius="${wheel_radius}" />
       </geometry>
-      <origin xyz="0 0.1175 0.034" rpy="1.5708 0 0" />
+      <origin xyz="0 0.1275 0.034" rpy="1.5708 0 0" />
       <material name="blue">
         <color rgba="0.0 0.0 1.0 1.0" />
@@ -40,5 +40,5 @@
         <cylinder length="${wheel_length}" radius="${wheel_radius}" />
       </geometry>
-      <origin xyz="0 -0.1175 0.034" rpy="1.5708 0 0" />
+      <origin xyz="0 -0.1275 0.034" rpy="1.5708 0 0" />
       <material name="blue">
         <color rgba="0.0 0.0 1.0 1.0" />

Commit message: redesign the hardware structure

File: my_robot_description/urdf/mobile_base.xacro (robot description, xacro)
@@ -13,5 +13,5 @@
         <box size="${base_length} ${base_width} ${base_height}" />
       </geometry>
-      <origin xyz="-0.105 0 0.0775" rpy="0 0 0" />
+      <origin xyz="-0.0675 0 0.0775" rpy="0 0 0" />
       <material name="semi_black">
         <color rgba="0 0 0 0.75" />
@@ -51,5 +51,5 @@
         <sphere radius="0.03" />
       </geometry>
-      <origin xyz="-0.21 0 0.03" rpy="0 0 0" />
+      <origin xyz="-0.135 0 0.03" rpy="0 0 0" />
       <material name="gray">
         <color rgba="0.5 0.5 0.5 1.0" />
@@ -100,5 +100,5 @@
     <parent link="base_link"/>
     <child link="imu_link"/>
-    <origin xyz="-0.105 0 0.0775" rpy="0 0 0"/>
+    <origin xyz="-0.045 0.03 0.0775" rpy="0 0 0"/>
   </joint>
 </robot>

Commit message: fix kinect RGB camera position

File: my_robot_description/urdf/mobile_base.xacro (robot description, xacro)
@@ -75,9 +75,10 @@
   </joint>
   <!-- Kinect Optical Frame (Z forward, X right, Y down) -->
+  <!-- Microsoft Kinect v1 offsets: RGB camera is 1.25cm right of center base (-0.0125 in Y) -->
   <link name="kinect_depth"/>
   <joint name="kinect_depth_joint" type="fixed">
     <parent link="kinect_link"/>
     <child link="kinect_depth"/>
-    <origin xyz="0 0 0" rpy="-1.5708 0 -1.5708"/>
+    <origin xyz="0 -0.0125 0" rpy="-1.5708 0 -1.5708"/>
   </joint>
   <joint name="left_wheel_joint" type="fixed">
